File: Hardware/relay_to_rs485/_autosave-relay_to_rs485.kicad_sch (KiCad schematic)
At the start: 46 parts, among them J1 Relay Inputs A to E connected, J2 RS485 Output Screw Terminal, J3 Screw_Terminal_InputGrounds, J4 Jack-DC, J5 UART OUT, Q1 IRLML6401, U1 ESP32-S3-WROOM-1, U2 MAX485E, U3 SMX1117MP-3.3

Commit message: More reworking of board
Addition of ZD1, MOSFET RP protection diode, reconfig of JP1 etc
Parts:
- added DZ1: 7.5 or 8.2, PCM_Diode_SMD_Handsoldering_AKL:D_SOD-123_Zener, symbol PCM_Diode_Zener_AKL:D_Zener_Generic
- J4: value Jack-DC -> Max 12VDC IN
- R3: value 10R -> 100R
- renumbered TP10 to TP10_B1, TP13 to TP13_3V3, TP14 to TP14_GND1, TP15 to TP15_VCC1, TP16 to TP16_TX1, TP17 to TP17_RX1, TP9 to TP9_A1
Connections:
- net GND: now also DZ1.2 (A)
- net VCC: now also DZ1.1 (K)
Changed lines of the file:
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@@
 	)
 	(junction
+		(at 34.29 35.56)
+		(diameter 0)
+		(color 0 0 0 0)
+	)
+	(junction
 		(at 46.99 27.94)
 		(diameter 0)
@@
 	)
 	(junction
-		(at 41.91 81.28)
+		(at 41.91 35.56)
 		(diameter 0)
 		(color 0 0 0 0)
 	)
 	(junction
-		(at 208.28 109.22)
+		(at 41.91 81.28)
 		(diameter 0)
 		(color 0 0 0 0)
 	)
 	(junction
-		(at 34.29 33.02)
+		(at 208.28 109.22)
 		(diameter 0)
 		(color 0 0 0 0)
@@
 	)
 	(junction
+		(at 41.91 27.94)
+		(diameter 0)
+		(color 0 0 0 0)
+	)
+	(junction
 		(at 146.05 54.61)
 		(diameter 0)
@@
 	(wire
 		(pts
-			(xy 34.29 33.02) (xy 48.26 33.02)
-		)
-		(stroke
-			(width 0)
-			(type default)
-		)
-	)
-	(wire
-		(pts
 			(xy 80.01 27.94) (xy 81.28 27.94)
 		)
@@
 	(wire
 		(pts
-			(xy 34.29 33.02) (xy 34.29 35.56)
+			(xy 34.29 29.21) (xy 34.29 35.56)
 		)
 		(stroke
@@
 	(wire
 		(pts
-			(xy 40.64 27.94) (xy 46.99 27.94)
-		)
-		(stroke
-			(width 0)
-			(type default)
-		)
-	)
-	(wire
-		(pts
 			(xy 41.91 96.52) (xy 62.23 96.52)
 		)
@@
 	(wire
 		(pts
-			(xy 34.29 29.21) (xy 34.29 33.02)
-		)
-		(stroke
-			(width 0)
-			(type default)
-		)
-	)
-	(wire
-		(pts
 			(xy 256.54 104.14) (xy 256.54 101.6)
 		)
@@
 	(wire
 		(pts
+			(xy 40.64 27.94) (xy 41.91 27.94)
+		)
+		(stroke
+			(width 0)
+			(type default)
+		)
+	)
+	(wire
+		(pts
 			(xy 146.05 142.24) (xy 146.05 143.51)
 		)
@@
 	(wire
 		(pts
-			(xy 48.26 35.56) (xy 48.26 33.02)
+			(xy 233.68 29.21) (xy 240.03 29.21)
 		)
 		(stroke
@@
 	(wire
 		(pts
-			(xy 233.68 29.21) (xy 240.03 29.21)
+			(xy 34.29 35.56) (xy 41.91 35.56)
 		)
 		(stroke
@@
 	(wire
 		(pts
-			(xy 53.34 35.56) (xy 48.26 35.56)
-		)
-		(stroke
-			(width 0)
-			(type default)
-		)
-	)
-	(wire
-		(pts
 			(xy 250.19 106.68) (xy 252.73 106.68)
 		)
@@
 	(wire
 		(pts
+			(xy 41.91 27.94) (xy 46.99 27.94)
+		)
+		(stroke
+			(width 0)
+			(type default)
+		)
+	)
+	(wire
+		(pts
+			(xy 41.91 35.56) (xy 53.34 35.56)
+		)
+		(stroke
+			(width 0)
+			(type default)
+		)
+	)
+	(wire
+		(pts
 			(xy 254 109.22) (xy 256.54 109.22)
 		)
@@
 		(dnp no)
 		(fields_autoplaced yes)
-		(property "Reference" "TP17"
+		(property "Reference" "TP17_RX1"
 			(at 241.3 30.1624 0)
 			(effects
@@
 			(project "relay_to_rs485"
 				(path "/3a402a89-4541-4a12-afbc-bb2d79b5f06e"
-					(reference "TP17")
+					(reference "TP17_RX1")
+					(unit 1)
+				)
+			)
+		)
+	)
+	(symbol
+		(lib_id "PCM_Diode_Zener_AKL:D_Zener_Generic")
+		(at 41.91 31.75 90)
+		(unit 1)
+		(exclude_from_sim no)
+		(in_bom yes)
+		(on_board yes)
+		(dnp no)
+		(fields_autoplaced yes)
+		(property "Reference" "DZ1"
+			(at 44.45 30.4799 90)
+			(effects
+				(font
+					(size 1.27 1.27)
+				)
+				(justify right)
+			)
+		)
+		(property "Value" "7.5 or 8.2"
+			(at 44.45 33.0199 90)
+			(effects
+				(font
+					(size 1.27 1.27)
+				)
+				(justify right)
+			)
+		)
+		(property "Footprint" "PCM_Diode_SMD_Handsoldering_AKL:D_SOD-123_Zener"
+			(at 41.91 31.75 0)
+			(effects
+				(font
+					(size 1.27 1.27)
+				)
+				(hide yes)
+			)
+		)
+		(property "Datasheet" "~"
+			(at 41.91 31.75 0)
+			(effects
+				(font
+					(size 1.27 1.27)
+				)
+				(hide yes)
+			)
+		)
+		(property "Description" "Zener diode, generic symbol, Alternate KiCAD Library"
+			(at 41.91 31.75 0)
+			(effects
+				(font
+					(size 1.27 1.27)
+				)
+				(hide yes)
+			)
+		)
+		(pin "2"
+		)
+		(pin "1"
+		)
+		(instances
+			(project ""
+				(path "/3a402a89-4541-4a12-afbc-bb2d79b5f06e"
+					(reference "DZ1")
 					(unit 1)
 				)
@@
 		(on_board yes)
 		(dnp no)
-		(property "Reference" "TP10"
+		(property "Reference" "TP10_B1"
 			(at 252.476 102.87 90)
 			(effects
@@
 			(project "relay_to_rs485"
 				(path "/3a402a89-4541-4a12-afbc-bb2d79b5f06e"
-					(reference "TP10")
+					(reference "TP10_B1")
 					(unit 1)
 				)
@@
 		(on_board yes)
 		(dnp no)
-		(property "Reference" "TP15"
+		(property "Reference" "TP15_VCC1"
 			(at 44.1324 24.13 0)
 			(effects
@@
 			(project "relay_to_rs485"
 				(path "/3a402a89-4541-4a12-afbc-bb2d79b5f06e"
-					(reference "TP15")
+					(reference "TP15_VCC1")
 					(unit 1)
 				)
@@
 		(dnp no)
 		(fields_autoplaced yes)
-		(property "Reference" "TP9"
+		(property "Reference" "TP9_A1"
 			(at 249.8725 96.52 90)
 			(effects
@@
 			(project "relay_to_rs485"
 				(path "/3a402a89-4541-4a12-afbc-bb2d79b5f06e"
-					(reference "TP9")
+					(reference "TP9_A1")
 					(unit 1)
 				)
@@
 		(dnp no)
 		(fields_autoplaced yes)
-		(property "Reference" "TP16"
-			(at 238.4425 21.59 90)
+		(property "Reference" "TP16_TX1"
+			(at 238.4425 20.32 90)
 			(effects
 				(font
@@
 		)
 		(property "Value" "~"
-			(at 239.7124 22.86 0)
+			(at 238.4425 21.59 90)
 			(effects
 				(font
 					(size 1.27 1.27)
 				)
-				(justify left)
 			)
 		)
@@
 			(project "relay_to_rs485"
 				(path "/3a402a89-4541-4a12-afbc-bb2d79b5f06e"
-					(reference "TP16")
+					(reference "TP16_TX1")
 					(unit 1)
 				)
@@
 			)
 		)
-		(property "Value" "Jack-DC"
+		(property "Value" "Max 12VDC IN"
 			(at 12.7 35.306 90)
 			(effects
@@
 		(on_board yes)
 		(dnp no)
-		(property "Reference" "TP13"
+		(property "Reference" "TP13_3V3"
 			(at 87.63 25.0824 0)
 			(effects
@@
 			(project "relay_to_rs485"
 				(path "/3a402a89-4541-4a12-afbc-bb2d79b5f06e"
-					(reference "TP13")
+					(reference "TP13_3V3")
 					(unit 1)
 				)
@@
 		(on_board yes)
 		(dnp no)
-		(property "Reference" "TP14"
+		(property "Reference" "TP14_GND1"
 			(at 149.86 139.3824 0)
 			(effects
@@
 			(project "relay_to_rs485"
 				(path "/3a402a89-4541-4a12-afbc-bb2d79b5f06e"
-					(reference "TP14")
+					(reference "TP14_GND1")
 					(unit 1)
 				)
@@
 			)
 		)
-		(property "Value" "10R"
+		(property "Value" "100R"
 			(at 28.448 26.162 0)
 			(effects

Commit message: More changes
Parts:
- C4: value 1uF -> 10uF
- R4, R5: value 680R -> 330R
Connections:
- net A renamed A+
- net B renamed B-
Other:
- moved on the sheet: D1, R1, R4, R5
